File: CAD/esprelay/io_driver.kicad_sch (KiCad schematic)
At the start: 2 parts, among them U3 ULN2003A

Commit message: Feat: Changed module to ESP12F
Connections:
- net LI2 is gone; now on net LI06: U3.10 (O7)
- net HPO4: no longer U3.12 (O5)
- net HI1 renamed HI06
- net HI2 renamed HI07
- net HO3 renamed HPO3
- net LI1 renamed LI06
- net LO3 renamed LP03
- net LO4 renamed HI05
- net HI05: no longer U3.4 (I4)
- new net LI05: U3.12 (O5)
- new net LPO4: U3.4 (I4)
Changed lines of the file:
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@@
-    (stroke (width 0) (type default))
-  )
-  (wire (pts (xy 116.84 90.17) (xy 116.84 92.71))
     (stroke (width 0) (type default))
   )
@@
     (stroke (width 0) (type default))
   )
-  (wire (pts (xy 137.16 90.17) (xy 137.16 92.71))
-    (stroke (width 0) (type default))
-  )
   (hierarchical_label "LRO2" (shape input) (at 116.84 85.09 180) (fields_autoplaced)
     (effects (font (size 1.27 1.27)) (justify right))
   )
-  (hierarchical_label "LI2" (shape input) (at 137.16 97.79 0) (fields_autoplaced)
+  (hierarchical_label "LI06" (shape input) (at 137.16 97.79 0) (fields_autoplaced)
     (effects (font (size 1.27 1.27)) (justify left))
   )
-  (hierarchical_label "HI1" (shape input) (at 116.84 95.25 180) (fields_autoplaced)
+  (hierarchical_label "HI05" (shape input) (at 116.84 92.71 180) (fields_autoplaced)
     (effects (font (size 1.27 1.27)) (justify right))
   )
-  (hierarchical_label "LI1" (shape input) (at 137.16 95.25 0) (fields_autoplaced)
+  (hierarchical_label "HI06" (shape input) (at 116.84 95.25 180) (fields_autoplaced)
+    (effects (font (size 1.27 1.27)) (justify right))
+  )
+  (hierarchical_label "LI06" (shape input) (at 137.16 95.25 0) (fields_autoplaced)
     (effects (font (size 1.27 1.27)) (justify left))
   )
@@
     (effects (font (size 1.27 1.27)) (justify right))
   )
-  (hierarchical_label "HI2" (shape input) (at 116.84 97.79 180) (fields_autoplaced)
+  (hierarchical_label "HI07" (shape input) (at 116.84 97.79 180) (fields_autoplaced)
     (effects (font (size 1.27 1.27)) (justify right))
   )
-  (hierarchical_label "LO4" (shape input) (at 116.84 90.17 180) (fields_autoplaced)
-    (effects (font (size 1.27 1.27)) (justify right))
-  )
-  (hierarchical_label "HO3" (shape input) (at 137.16 87.63 0) (fields_autoplaced)
+  (hierarchical_label "HPO3" (shape input) (at 137.16 87.63 0) (fields_autoplaced)
     (effects (font (size 1.27 1.27)) (justify left))
   )
-  (hierarchical_label "LO3" (shape input) (at 116.84 87.63 180) (fields_autoplaced)
+  (hierarchical_label "LP03" (shape input) (at 116.84 87.63 180) (fields_autoplaced)
     (effects (font (size 1.27 1.27)) (justify right))
   )
@@
     (effects (font (size 1.27 1.27)) (justify left))
   )
+  (hierarchical_label "LI05" (shape input) (at 137.16 92.71 0) (fields_autoplaced)
+    (effects (font (size 1.27 1.27)) (justify left))
+  )
